File: KiCAD/hexpansion-L80.kicad_pcb (KiCad board)
At the start: 2 copper layers, 40.1 x 36.4 mm, 22 parts, among them J1 Hexpansion-Connector, J2 Conn_Coaxial, Q1 BC847, U1 L80RE-M37, U2 M24C16-RMN6TP

Commit message: rotated LEDs, fixed footprint sizing and regenerated production files
Parts:
- D1: value YELLOW -> WHITE
- moved C1 0.07 mm to (167.1, 110.8)
- turned D1 to 180 degrees
- turned D2 to 180 degrees
Connections:
- D1 pad 1: /LS_C -> Net-(D1-K)
- D1 pad 2: Net-(D1-A) -> /LS_C
- D2 pad 1: /LS_D -> Net-(D2-K)
- D2 pad 2: Net-(D2-A) -> /LS_D
- R3 pad 2: Net-(D1-A) -> Net-(D1-K)
- R4 pad 2: Net-(D2-A) -> Net-(D2-K)
Routing:
- net Net-(D2-K): track 0.00 -> 1.15 mm
- net Net-(D2-A): track 1.15 -> 0.00 mm
- net Net-(D1-K): track 0.00 -> 1.15 mm
- net Net-(D1-A): track 1.15 -> 0.00 mm
